Commit message: add inertia to urdf links

File: src/urdf_try_moving/urdf/v3_approx_xacro.urdf (robot description, URDF)
Before this commit: robot adam, 5 links, 4 joints
Joints:
- joint tray_joint: origin xyz=${tray_length / 2 - holder_radius * 2} ${tray_width / 2 - holder_radius * 2} ${(holder_length + tray_height) / 2} -> xyz=${tray_length / 2 - holder_radius * 2} ${tray_width / 2 - holder_radius * 2} ${holder_length / 2 - tray_height / 2}

Commit message: integrate urdf with lidar

File: src/urdf_try_moving/urdf/v3_approx_xacro.urdf (robot description, URDF)
Before this commit: robot adam, 5 links, 4 joints
Joints:
- joint caster_wheel_joint: type planar -> fixed

Commit message: fix robot rotation

File: src/urdf_try_moving/urdf/v3_approx_xacro.urdf (robot description, URDF)
Before this commit: robot adam, 5 links, 4 joints
Joints:
- joint caster_wheel_joint: type fixed -> continuous
