Commit message: fixed robot slow motion during nav2 navigation

File: src/neu_lidar/model/v3_approx_xacro.urdf (robot description, URDF)
Before this commit: robot adam, 5 links, 4 joints
Links:
- removed link tray
Joints:
- removed joint tray_joint

Commit message: working map no imu

File: src/neu_lidar/model/v3_approx_xacro.urdf (robot description, URDF)
Before this commit: robot adam, 4 links, 3 joints
Joints:
- joint lidar_joint: origin xyz=0 0 ${(lidar_length + body_height) / 2} -> xyz=0 0 ${(lidar_length + body_height) / 2} rpy=0 0 ${22 / 7}

Commit message: separate urdf into multiple files

File: src/neu_lidar/model/v3_approx_xacro.urdf (robot description, URDF)
Before this commit: robot adam, 4 links, 3 joints
Links:
- removed link base_link
- removed link body
- removed link caster_wheel
- removed link lidar
Joints:
- removed joint body_joint
- removed joint caster_wheel_joint
- removed joint lidar_joint
